File: pcb/leany.kicad_sch (KiCad schematic)
At the start: 42 parts, among them J1 ST7735S, J2 SWD, Q1 AO3401A, SW1 ZERO, SW2 HOLD, SW3 RESET, SW4 FLASH, U1 STM32F103C8Tx, U2 CH340N, U3 BMI270, Y1 8MHz

Commit message: update capacitors BOM
Parts:
- C10, C12, C2, C25, C26, C6, C7, C8, C9: LCSC C14663 -> C1525
- C3, C4: LCSC C1648 -> C1554
- C5: LCSC C15849 -> C52923
Changed lines of the file:
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@@
 			)
 		)
-		(property "LCSC" "C14663"
+		(property "LCSC" "C1525"
 			(at 161.29 50.8 0)
 			(effects
@@
 			)
 		)
-		(property "LCSC" "C1648"
+		(property "LCSC" "C1554"
 			(at 91.44 83.82 0)
 			(effects
@@
 			)
 		)
-		(property "LCSC" "C14663"
+		(property "LCSC" "C1525"
 			(at 199.39 99.06 0)
 			(effects
@@
 			)
 		)
-		(property "LCSC" "C14663"
+		(property "LCSC" "C1525"
 			(at 66.04 46.99 0)
 			(effects
@@
 			)
 		)
-		(property "LCSC" "C14663"
+		(property "LCSC" "C1525"
 			(at 232.41 31.75 0)
 			(effects
@@
 			)
 		)
-		(property "LCSC" "C15849"
+		(property "LCSC" "C52923"
 			(at 109.22 68.58 0)
 			(effects
@@
 			)
 		)
-		(property "LCSC" "C14663"
+		(property "LCSC" "C1525"
 			(at 238.76 31.75 0)
 			(effects
@@
 			)
 		)
-		(property "LCSC" "C14663"
+		(property "LCSC" "C1525"
 			(at 154.94 50.8 0)
 			(effects
@@
 			)
 		)
-		(property "LCSC" "C1648"
+		(property "LCSC" "C1554"
 			(at 91.44 76.2 0)
 			(effects
@@
 			)
 		)
-		(property "LCSC" "C14663"
+		(property "LCSC" "C1525"
 			(at 142.24 50.8 0)
 			(effects
@@
 			)
 		)
-		(property "LCSC" "C14663"
+		(property "LCSC" "C1525"
 			(at 148.59 50.8 0)
 			(effects
@@
 			)
 		)
-		(property "LCSC" "C14663"
+		(property "LCSC" "C1525"
 			(at 207.01 99.06 0)
 			(effects

Commit message: fix capacitors silkscreen issues
Parts:
- C10, C12, C2, C25, C26, C3, C4, C5, C6, C7, C8, C9: footprint Capacitor_SMD:C_0402_1005Metric -> leany_footprints:C_0402_1005Metric
Changed lines of the file:
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@@
 			)
 		)
-		(property "Footprint" "Capacitor_SMD:C_0402_1005Metric"
+		(property "Footprint" "leany_footprints:C_0402_1005Metric"
 			(at 161.29 50.8 0)
 			(effects
@@
 			)
 		)
-		(property "Footprint" "Capacitor_SMD:C_0402_1005Metric"
+		(property "Footprint" "leany_footprints:C_0402_1005Metric"
 			(at 91.44 83.82 0)
 			(effects
@@
 			)
 		)
-		(property "Footprint" "Capacitor_SMD:C_0402_1005Metric"
+		(property "Footprint" "leany_footprints:C_0402_1005Metric"
 			(at 199.39 99.06 0)
 			(effects
@@
 			)
 		)
-		(property "Footprint" "Capacitor_SMD:C_0402_1005Metric"
+		(property "Footprint" "leany_footprints:C_0402_1005Metric"
 			(at 66.04 46.99 0)
 			(effects
@@
 			)
 		)
-		(property "Footprint" "Capacitor_SMD:C_0402_1005Metric"
+		(property "Footprint" "leany_footprints:C_0402_1005Metric"
 			(at 232.41 31.75 0)
 			(effects
@@
 			)
 		)
-		(property "Footprint" "Capacitor_SMD:C_0402_1005Metric"
+		(property "Footprint" "leany_footprints:C_0402_1005Metric"
 			(at 109.22 68.58 0)
 			(effects
@@
 			)
 		)
-		(property "Footprint" "Capacitor_SMD:C_0402_1005Metric"
+		(property "Footprint" "leany_footprints:C_0402_1005Metric"
 			(at 238.76 31.75 0)
 			(effects
@@
 			)
 		)
-		(property "Footprint" "Capacitor_SMD:C_0402_1005Metric"
+		(property "Footprint" "leany_footprints:C_0402_1005Metric"
 			(at 154.94 50.8 0)
 			(effects
@@
 			)
 		)
-		(property "Footprint" "Capacitor_SMD:C_0402_1005Metric"
+		(property "Footprint" "leany_footprints:C_0402_1005Metric"
 			(at 91.44 76.2 0)
 			(effects
@@
 			)
 		)
-		(property "Footprint" "Capacitor_SMD:C_0402_1005Metric"
+		(property "Footprint" "leany_footprints:C_0402_1005Metric"
 			(at 142.24 50.8 0)
 			(effects
@@
 			)
 		)
-		(property "Footprint" "Capacitor_SMD:C_0402_1005Metric"
+		(property "Footprint" "leany_footprints:C_0402_1005Metric"
 			(at 148.59 50.8 0)
 			(effects
@@
 			)
 		)
-		(property "Footprint" "Capacitor_SMD:C_0402_1005Metric"
+		(property "Footprint" "leany_footprints:C_0402_1005Metric"
 			(at 207.01 99.06 0)
 			(effects

Commit message: fix resistors silkscreen issues
Parts:
- R1, R10, R11, R12, R13, R14, R15, R2, R3, R7, R8, R9: footprint Resistor_SMD:R_0402_1005Metric -> leany_footprints:R_0402_1005Metric
Changed lines of the file:
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@@
 			)
 		)
-		(property "Footprint" "Resistor_SMD:R_0402_1005Metric"
+		(property "Footprint" "leany_footprints:R_0402_1005Metric"
 			(at 252.73 121.92 0)
 			(effects
@@
 			)
 		)
-		(property "Footprint" "Resistor_SMD:R_0402_1005Metric"
+		(property "Footprint" "leany_footprints:R_0402_1005Metric"
 			(at 38.1 52.07 0)
 			(effects
@@
 			)
 		)
-		(property "Footprint" "Resistor_SMD:R_0402_1005Metric"
+		(property "Footprint" "leany_footprints:R_0402_1005Metric"
 			(at 40.64 52.07 0)
 			(effects
@@
 			)
 		)
-		(property "Footprint" "Resistor_SMD:R_0402_1005Metric"
+		(property "Footprint" "leany_footprints:R_0402_1005Metric"
 			(at 200.66 52.07 0)
 			(effects
@@
 			)
 		)
-		(property "Footprint" "Resistor_SMD:R_0402_1005Metric"
+		(property "Footprint" "leany_footprints:R_0402_1005Metric"
 			(at 252.73 104.14 0)
 			(effects
@@
 			)
 		)
-		(property "Footprint" "Resistor_SMD:R_0402_1005Metric"
+		(property "Footprint" "leany_footprints:R_0402_1005Metric"
 			(at 196.85 116.84 0)
 			(effects
@@
 			)
 		)
-		(property "Footprint" "Resistor_SMD:R_0402_1005Metric"
+		(property "Footprint" "leany_footprints:R_0402_1005Metric"
 			(at 59.69 86.36 0)
 			(effects
@@
 			)
 		)
-		(property "Footprint" "Resistor_SMD:R_0402_1005Metric"
+		(property "Footprint" "leany_footprints:R_0402_1005Metric"
 			(at 115.57 60.96 0)
 			(effects
@@
 			)
 		)
-		(property "Footprint" "Resistor_SMD:R_0402_1005Metric"
+		(property "Footprint" "leany_footprints:R_0402_1005Metric"
 			(at 196.85 114.3 0)
 			(effects
@@
 			)
 		)
-		(property "Footprint" "Resistor_SMD:R_0402_1005Metric"
+		(property "Footprint" "leany_footprints:R_0402_1005Metric"
 			(at 104.14 80.01 0)
 			(effects
@@
 			)
 		)
-		(property "Footprint" "Resistor_SMD:R_0402_1005Metric"
+		(property "Footprint" "leany_footprints:R_0402_1005Metric"
 			(at 41.91 138.43 0)
 			(effects
@@
 			)
 		)
-		(property "Footprint" "Resistor_SMD:R_0402_1005Metric"
+		(property "Footprint" "leany_footprints:R_0402_1005Metric"
 			(at 100.33 104.14 0)
 			(effects
