File: pcb/leany.kicad_pcb (KiCad board)
At the start: 4 copper layers, 80.4 x 49.3 mm, 83 parts, among them J1 ST7735S, J2 SWD, J3 USB C, J4 BATT, Q1 AO3401A, Q2 AO3400A, Q3 AO3401A, Q4 AO3401A, Q5 PT8810, SW1 ZERO, SW2 HOLD, SW3 RESET, SW4 BOOT, SW5 POWER, U1 STM32F103C8Tx, U2 CH340N, U3 ICM-42688-P, U4 BQ25619, U5 AP2112K-3.3, U6 DW01A, Y1 8MHz

Commit message: feat: place and route external eeprom (#90)
Parts:
- removed R23, R24: 4k7, leany_footprints:R_0402_1005Metric
- added C27: 100n, leany_footprints:C_0402_1005Metric, F.Cu at (145.9, 89.4)
- added R27: 10k, leany_footprints:R_0402_1005Metric, F.Cu at (145.4, 87.9)
- added R28: 4k7, leany_footprints:R_0402_1005Metric, F.Cu at (132.6, 91.7)
- added R29: 4k7, leany_footprints:R_0402_1005Metric, F.Cu at (130.6, 91.7)
- added U7: 24C02S, Package_TO_SOT_SMD:SOT-23-5, F.Cu at (142.8, 88.5)
Connections:
- net CHG_SCL renamed I2C_SCL
- net CHG_SDA renamed I2C_SDA
- U1 pad 45: unconnected-(U1-PB8-Pad45) -> /EEPROM_WP
Routing:
- net /EEPROM_WP: track 0.00 -> 23.0 mm
- net I2C_SDA: track 45.8 -> 57.9 mm, vias 4 -> 5
- net I2C_SCL: track 43.9 -> 53.5 mm
- net +3V3: track 37.4 -> 37.6 mm, vias 30 -> 31
- net GND: vias 80 -> 82
Other:
- board text added: "${TITLE}"
- board text added: "rev. ${REVISION}"
- board text removed: "Leany"
- board text removed: "rev. 0.3"
