File: pcb/leany.kicad_pcb (KiCad board)
At the start: 4 copper layers, 80.4 x 49.3 mm, 86 parts, among them J1 ST7735S, J2 SWD, J3 USB C, J4 BATT, Q1 AO3401A, Q2 AO3400A, Q3 AO3401A, Q4 AO3401A, Q5 PT8810, SW1 ZERO, SW2 HOLD, SW3 RESET, SW4 BOOT, SW5 POWER, U1 STM32F103C8Tx, U2 CH340N, U3 ICM-42688-P, U4 BQ25619, U5 AP2112K-3.3, U6 DW01A, U7 24C02S, Y1 8MHz

Commit message: refactor: improve STM32 decoupling (#90)
Parts:
- added C29: 100n, leany_footprints:C_0402_1005Metric, F.Cu at (167.1, 99.0)
- added C30: 4.7u, leany_footprints:C_0402_1005Metric, F.Cu at (160.0, 87.1)
- added C31: 1u, leany_footprints:C_0402_1005Metric, F.Cu at (155.2, 94.2)
- added C32: 10n, leany_footprints:C_0402_1005Metric, F.Cu at (155.2, 95.2)
- moved C9 14.8 mm to (169.5, 90.2), turned to -90 degrees
- moved C7 1.00 mm to (160.0, 86.1)
Routing:
- net GND: track 23.1 -> 3.97 mm
- net +3V3: track 37.6 -> 39.5 mm
- net /ST7735S_BL: track 25.6 -> 27.2 mm
- net /EEPROM_WP: track 23.0 -> 23.7 mm

Commit message: refactor: beef up the crystal load capacitors (#90)
Parts:
- C3, C4: value 20p -> 33p
Changed lines of the file:
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@@
 			)
 		)
-		(property "Value" "20p"
+		(property "Value" "33p"
 			(at -0.66 1.1925 0)
 			(layer "F.Fab")
@@
 			)
 		)
-		(property "LCSC" "C1554"
+		(property "LCSC" "C1562"
 			(at 0 0 0)
 			(unlocked yes)
@@
 			)
 		)
-		(property "Value" "20p"
+		(property "Value" "33p"
 			(at 0 -1.16 0)
 			(layer "F.Fab")
@@
 			)
 		)
-		(property "LCSC" "C1554"
+		(property "LCSC" "C1562"
 			(at 0 0 0)
 			(unlocked yes)

Commit message: refactor: update wire stripping information (#90)
Other:
- board text added: "0.14"
- board text added: "0.34"
- board text added: "22"
- board text added: "26"
- board text added: "4mm"
- board text added: "5.5mm"
- board text removed: "0.2"
- board text removed: "0.75"
- board text removed: "18"
- board text removed: "24"
- board text removed: "7mm"
- board text removed: "9mm"
Changed lines of the file:
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@@
 	(gr_line
 		(start 127.53 125.16)
-		(end 136.53 125.16)
+		(end 133.03 125.16)
 		(stroke
 			(width 0.2)
-			(type default)
-		)
-		(layer "B.SilkS")
-	)
-	(gr_line
-		(start 134.53 124.66)
-		(end 134.53 125.66)
+			(type solid)
+		)
+		(layer "B.SilkS")
+	)
+	(gr_line
+		(start 131.53 124.66)
+		(end 131.53 125.66)
 		(stroke
 			(width 0.2)
-			(type default)
-		)
-		(layer "B.SilkS")
-	)
-	(gr_line
-		(start 136.53 124.46)
-		(end 136.53 125.86)
+			(type solid)
+		)
+		(layer "B.SilkS")
+	)
+	(gr_line
+		(start 133.03 124.46)
+		(end 133.03 125.86)
 		(stroke
 			(width 0.2)
-			(type default)
+			(type solid)
 		)
 		(layer "B.SilkS")
@@
 		)
 	)
-	(gr_text "7mm"
+	(gr_text "4mm"
 		(at 133.33 120.46 0)
 		(layer "B.SilkS")
@@
 		)
 	)
-	(gr_text "9mm"
+	(gr_text "5.5mm"
 		(at 133.33 122.96 0)
 		(layer "B.SilkS")
@@
 		)
 	)
-	(gr_text "24"
+	(gr_text "26"
 		(at 140.43 120.46 0)
 		(layer "B.SilkS")
@@
 		)
 	)
-	(gr_text "18"
+	(gr_text "22"
 		(at 140.43 122.96 0)
 		(layer "B.SilkS")
@@
 		)
 	)
-	(gr_text "0.2"
+	(gr_text "0.14"
 		(at 147.753809 120.46 0)
 		(layer "B.SilkS")
@@
 		)
 	)
-	(gr_text "0.75"
+	(gr_text "0.34"
 		(at 148.23 122.96 0)
 		(layer "B.SilkS")

Commit message: refactor: cleanup routing (#90)
Routing:
- net Net-(U4-~{QON}): track 38.9 -> 43.9 mm
- net /ST7735S_BL: track 27.2 -> 25.7 mm
- net Net-(Q3-D): track 12.0 -> 13.5 mm
- net /ST7735S_CS: track 16.8 -> 17.7 mm

Commit message: feat: add mounting holes (#90)
Parts:
- added H1: MountingHole, MountingHole:MountingHole_3.2mm_M3, F.Cu at (181.3, 87.3)
- added H2: MountingHole, MountingHole:MountingHole_3.2mm_M3, F.Cu at (181.3, 122.0)
- added H3: MountingHole, MountingHole:MountingHole_3.2mm_M3, F.Cu at (120.2, 122.0)
- added H4: MountingHole, MountingHole:MountingHole_3.2mm_M3, F.Cu at (120.8, 89.7)
