File: pcb/power_management.kicad_sch (KiCad schematic)
At the start: 41 parts, among them J3 USB C, J4 BATT, Q2 AO3400A, Q3 AO3401A, Q4 AO3401A, Q5 PT8810, SW5 POWER, U4 BQ25619, U5 AP2112K-3.3, U6 DW01A

Commit message: ci: optimise kicad CI (#106)
Parts:
- C14, C15, C16, C17, C20, C21, C22, C23, C28: symbol Device:C_Small -> leany-symbols:C_Small
Changed lines of the file:
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@@
 	)
 	(symbol
-		(lib_id "Device:C_Small")
+		(lib_id "leany-symbols:C_Small")
 		(at 171.45 123.19 0)
 		(mirror y)
@@
 	)
 	(symbol
-		(lib_id "Device:C_Small")
+		(lib_id "leany-symbols:C_Small")
 		(at 213.36 41.91 0)
 		(unit 1)
@@
 	)
 	(symbol
-		(lib_id "Device:C_Small")
+		(lib_id "leany-symbols:C_Small")
 		(at 113.03 41.91 0)
 		(unit 1)
@@
 	)
 	(symbol
-		(lib_id "Device:C_Small")
+		(lib_id "leany-symbols:C_Small")
 		(at 166.37 57.15 0)
 		(unit 1)
@@
 	)
 	(symbol
-		(lib_id "Device:C_Small")
+		(lib_id "leany-symbols:C_Small")
 		(at 218.44 41.91 0)
 		(unit 1)
@@
 	)
 	(symbol
-		(lib_id "Device:C_Small")
+		(lib_id "leany-symbols:C_Small")
 		(at 208.28 41.91 0)
 		(unit 1)
@@
 	)
 	(symbol
-		(lib_id "Device:C_Small")
+		(lib_id "leany-symbols:C_Small")
 		(at 161.29 39.37 0)
 		(unit 1)
@@
 	)
 	(symbol
-		(lib_id "Device:C_Small")
+		(lib_id "leany-symbols:C_Small")
 		(at 241.3 41.91 0)
 		(unit 1)
@@
 	)
 	(symbol
-		(lib_id "Device:C_Small")
+		(lib_id "leany-symbols:C_Small")
 		(at 162.56 68.58 0)
 		(unit 1)

Commit message: feat: place and route external eeprom (#90)
Parts:
- removed R23, R24: 4k7, leany_footprints:R_0402_1005Metric, symbol Device:R_Small
Connections:
- net CHG_SCL renamed I2C_SCL
- net CHG_SDA renamed I2C_SDA
